Commit message: add ground plane to URDF

File: ur_e_description/urdf/ur3e_joint_limited_robot.urdf.xacro (robot description, xacro)
@@ -24,6 +24,28 @@
   <joint name="world_joint" type="fixed">
     <parent link="world" />
-    <child link = "base_link" />
-    <origin xyz="0.0 0.0 0.0" rpy="0.0 0.0 0.0" />
+    <child link = "ground_plane_box" />
+    <origin xyz="0.0 0.0 0.25" rpy="0.0 0.0 0.0" />
+  </joint>
+  <link name="ground_plane_box">
+    <visual>
+      <origin xyz="0 0 0" rpy="0 0 0"/>
+      <geometry>
+        <box size="1.0 1.0 0.5"/>
+      </geometry>
+      <material name="Grey">
+        <color rgba="0.7 0.7 0.7 1.0"/>
+      </material>
+    </visual>
+    <collision>
+      <origin xyz="0 0 0" rpy="0 0 0"/>
+      <geometry>
+        <box size="1.0 1.0 0.5"/>
+      </geometry>
+    </collision>
+  </link>
+  <joint name="ground_plane_box_joint" type="fixed">
+    <parent link="ground_plane_box" />
+    <child link="base_link" />
+    <origin xyz="0 0 0.25" rpy="0 0 0" />
   </joint>
 </robot>

File: ur_e_description/urdf/ur3e_robot.urdf.xacro (robot description, xacro)
@@ -16,6 +16,28 @@
   <joint name="world_joint" type="fixed">
     <parent link="world" />
-    <child link = "base_link" />
-    <origin xyz="0.0 0.0 0.0" rpy="0.0 0.0 0.0" />
+    <child link = "ground_plane_box" />
+    <origin xyz="0.0 0.0 0.25" rpy="0.0 0.0 0.0" />
+  </joint>
+  <link name="ground_plane_box">
+    <visual>
+      <origin xyz="0 0 0" rpy="0 0 0"/>
+      <geometry>
+        <box size="1.0 1.0 0.5"/>
+      </geometry>
+      <material name="Grey">
+        <color rgba="0.7 0.7 0.7 1.0"/>
+      </material>
+    </visual>
+    <collision>
+      <origin xyz="0 0 0" rpy="0 0 0"/>
+      <geometry>
+        <box size="1.0 1.0 0.5"/>
+      </geometry>
+    </collision>
+  </link>
+  <joint name="ground_plane_box_joint" type="fixed">
+    <parent link="ground_plane_box" />
+    <child link="base_link" />
+    <origin xyz="0 0 0.25" rpy="0 0 0" />
   </joint>
 </robot>

Commit message: fix baseplane

File: ur_e_description/urdf/ur3e_joint_limited_robot.urdf.xacro (robot description, xacro)
@@ -24,6 +24,11 @@
   <joint name="world_joint" type="fixed">
     <parent link="world" />
+    <child link = "base_link" />
+    <origin xyz="0.0 0.0 0.0" rpy="0.0 0.0 0.0" />
+  </joint>
+  <joint name="ground_joint" type="fixed">
+    <parent link="world" />
     <child link = "ground_plane_box" />
-    <origin xyz="0.0 0.0 0.25" rpy="0.0 0.0 0.0" />
+    <origin xyz="0.0 0.0 -0.26" rpy="0.0 0.0 0.0" />
   </joint>
   <link name="ground_plane_box">
@@ -44,8 +49,3 @@
     </collision>
   </link>
-  <joint name="ground_plane_box_joint" type="fixed">
-    <parent link="ground_plane_box" />
-    <child link="base_link" />
-    <origin xyz="0 0 0.25" rpy="0 0 0" />
-  </joint>
 </robot>

File: ur_e_description/urdf/ur3e_robot.urdf.xacro (robot description, xacro)
@@ -16,6 +16,11 @@
   <joint name="world_joint" type="fixed">
     <parent link="world" />
+    <child link = "base_link" />
+    <origin xyz="0.0 0.0 0.0" rpy="0.0 0.0 0.0" />
+  </joint>
+  <joint name="ground_joint" type="fixed">
+    <parent link="world" />
     <child link = "ground_plane_box" />
-    <origin xyz="0.0 0.0 0.25" rpy="0.0 0.0 0.0" />
+    <origin xyz="0.0 0.0 -0.26" rpy="0.0 0.0 0.0" />
   </joint>
   <link name="ground_plane_box">
@@ -36,8 +41,3 @@
     </collision>
   </link>
-  <joint name="ground_plane_box_joint" type="fixed">
-    <parent link="ground_plane_box" />
-    <child link="base_link" />
-    <origin xyz="0 0 0.25" rpy="0 0 0" />
-  </joint>
 </robot>

Commit message: add ground plane box from baseplane branch

File: ur_e_description/urdf/ur3e_joint_limited_robot.urdf.xacro (robot description, xacro)
@@ -31,3 +31,25 @@
     <origin xyz="0.0 0.0 0.0" rpy="0.0 0.0 0.0" />
   </joint>
+  <joint name="ground_joint" type="fixed">
+    <parent link="world" />
+    <child link = "ground_plane_box" />
+    <origin xyz="0.0 0.0 -0.26" rpy="0.0 0.0 0.0" />
+  </joint>
+  <link name="ground_plane_box">
+    <visual>
+      <origin xyz="0 0 0" rpy="0 0 0"/>
+      <geometry>
+        <box size="1.0 1.0 0.5"/>
+      </geometry>
+      <material name="Grey">
+        <color rgba="0.7 0.7 0.7 1.0"/>
+      </material>
+    </visual>
+    <collision>
+      <origin xyz="0 0 0" rpy="0 0 0"/>
+      <geometry>
+        <box size="1.0 1.0 0.5"/>
+      </geometry>
+    </collision>
+  </link>
 </robot>

File: ur_e_description/urdf/ur3e_robot.urdf.xacro (robot description, xacro)
@@ -19,3 +19,25 @@
     <origin xyz="0.0 0.0 0.0" rpy="0.0 0.0 0.0" />
   </joint>
+  <joint name="ground_joint" type="fixed">
+    <parent link="world" />
+    <child link = "ground_plane_box" />
+    <origin xyz="0.0 0.0 -0.26" rpy="0.0 0.0 0.0" />
+  </joint>
+  <link name="ground_plane_box">
+    <visual>
+      <origin xyz="0 0 0" rpy="0 0 0"/>
+      <geometry>
+        <box size="1.0 1.0 0.5"/>
+      </geometry>
+      <material name="Grey">
+        <color rgba="0.7 0.7 0.7 1.0"/>
+      </material>
+    </visual>
+    <collision>
+      <origin xyz="0 0 0" rpy="0 0 0"/>
+      <geometry>
+        <box size="1.0 1.0 0.5"/>
+      </geometry>
+    </collision>
+  </link>
 </robot>

Commit message: add another collision box to avoid strange moveit plans

File: ur_e_description/urdf/ur3e_joint_limited_robot.urdf.xacro (robot description, xacro)
@@ -53,3 +53,25 @@
     </collision>
   </link>
+  <joint name="ground_joint2" type="fixed">
+    <parent link="ground_plane_box" />
+    <child link = "ground_plane_box_board" />
+    <origin xyz="0.0 0.4 0.3" rpy="0.0 0.0 0.0" />
+  </joint>
+  <link name="ground_plane_box_board">
+    <visual>
+      <origin xyz="0 0 0" rpy="0 0 0"/>
+      <geometry>
+        <box size="0.4 0.4 0.15"/>
+      </geometry>
+      <material name="Grey">
+        <color rgba="0.7 0.7 0.7 1.0"/>
+      </material>
+    </visual>
+    <collision>
+      <origin xyz="0 0 0" rpy="0 0 0"/>
+      <geometry>
+        <box size="0.4 0.4 0.15"/>
+      </geometry>
+    </collision>
+  </link>
 </robot>

Commit message: increase chessboard collider height

File: ur_e_description/urdf/ur3e_joint_limited_robot.urdf.xacro (robot description, xacro)
@@ -56,5 +56,5 @@
     <parent link="ground_plane_box" />
     <child link = "ground_plane_box_board" />
-    <origin xyz="0.0 0.4 0.3" rpy="0.0 0.0 0.0" />
+    <origin xyz="0.0 0.4 0.325" rpy="0.0 0.0 0.0" />
   </joint>
   <link name="ground_plane_box_board">
