Commit message: add gripper to the URDF

File: ur_description/urdf/inc/ur3e_macro.xacro (robot description, xacro)
@@ -40,4 +40,6 @@
       safety_k_position="${safety_k_position}"
     />
+    <!-- rh_p12_rn_a -->
+    <xacro:include filename="$(find rh_p12_rn_a_description)/urdf/rh_p12_rn_a.xacro" />
   </xacro:macro>
 </robot>

File: ur_gazebo/urdf/ur.xacro (robot description, xacro)
@@ -69,3 +69,52 @@
   <!-- rh_p12_rn_a -->
   <xacro:include filename="$(find rh_p12_rn_a_description)/urdf/rh_p12_rn_a.xacro" />
+  <!-- camera -->
+  <xacro:include filename="$(find mogi_chess_gazebo)/urdf/camera.xacro" />
+  <!-- touch sensor -->
+  <xacro:include filename="$(find mogi_chess_gazebo)/urdf/touch.xacro" />
+  <!-- add ground plane box TODO: this should be moved to another xacro -->
+  <joint name="ground_joint" type="fixed">
+    <parent link="world" />
+    <child link = "ground_plane_box" />
+    <origin xyz="0.0 0.0 -0.26" rpy="0.0 0.0 0.0" />
+  </joint>
+  <link name="ground_plane_box">
+    <visual>
+      <origin xyz="0 0 0" rpy="0 0 0"/>
+      <geometry>
+        <box size="1.0 1.0 0.5"/>
+      </geometry>
+      <material name="Grey">
+        <color rgba="0.7 0.7 0.7 1.0"/>
+      </material>
+    </visual>
+    <collision>
+      <origin xyz="0 0 0" rpy="0 0 0"/>
+      <geometry>
+        <box size="1.0 1.0 0.5"/>
+      </geometry>
+    </collision>
+  </link>
+  <joint name="ground_joint2" type="fixed">
+    <parent link="ground_plane_box" />
+    <child link = "ground_plane_box_board" />
+    <origin xyz="0.0 0.4 0.325" rpy="0.0 0.0 0.0" />
+  </joint>
+  <link name="ground_plane_box_board">
+    <visual>
+      <origin xyz="0 0 0" rpy="0 0 0"/>
+      <geometry>
+        <box size="0.4 0.4 0.15"/>
+      </geometry>
+      <material name="Grey">
+        <color rgba="0.7 0.7 0.7 1.0"/>
+      </material>
+    </visual>
+    <collision>
+      <origin xyz="0 0 0" rpy="0 0 0"/>
+      <geometry>
+        <box size="0.4 0.4 0.15"/>
+      </geometry>
+    </collision>
+  </link>
 </robot>

Commit message: add ground plane box to the urdf

File: ur_description/urdf/inc/ur3e_macro.xacro (robot description, xacro)
@@ -40,6 +40,62 @@
       safety_k_position="${safety_k_position}"
     />
+    <!-- world link -->
+    <link name="world"/>
+    <joint name="world_joint" type="fixed">
+      <parent link="world"/>
+      <child link="base_link"/>
+      <origin xyz="0 0 0" rpy="0 0 0"/>
+    </joint>
     <!-- rh_p12_rn_a -->
     <xacro:include filename="$(find rh_p12_rn_a_description)/urdf/rh_p12_rn_a.xacro" />
+    <!-- camera -->
+    <xacro:include filename="$(find mogi_chess_gazebo)/urdf/camera.xacro" />
+    <!-- touch sensor -->
+    <xacro:include filename="$(find mogi_chess_gazebo)/urdf/touch.xacro" />
+    <!-- add ground plane box TODO: this should be moved to another xacro -->
+    <joint name="ground_joint" type="fixed">
+      <parent link="world" />
+      <child link = "ground_plane_box" />
+      <origin xyz="0.0 0.0 -0.26" rpy="0.0 0.0 0.0" />
+    </joint>
+    <link name="ground_plane_box">
+      <visual>
+        <origin xyz="0 0 0" rpy="0 0 0"/>
+        <geometry>
+          <box size="1.0 1.0 0.5"/>
+        </geometry>
+        <material name="Grey">
+          <color rgba="0.7 0.7 0.7 1.0"/>
+        </material>
+      </visual>
+      <collision>
+        <origin xyz="0 0 0" rpy="0 0 0"/>
+        <geometry>
+          <box size="1.0 1.0 0.5"/>
+        </geometry>
+      </collision>
+    </link>
+    <joint name="ground_joint2" type="fixed">
+      <parent link="ground_plane_box" />
+      <child link = "ground_plane_box_board" />
+      <origin xyz="0.0 0.4 0.325" rpy="0.0 0.0 0.0" />
+    </joint>
+    <link name="ground_plane_box_board">
+      <visual>
+        <origin xyz="0 0 0" rpy="0 0 0"/>
+        <geometry>
+          <box size="0.4 0.4 0.15"/>
+        </geometry>
+        <material name="Grey">
+          <color rgba="0.7 0.7 0.7 1.0"/>
+        </material>
+      </visual>
+      <collision>
+        <origin xyz="0 0 0" rpy="0 0 0"/>
+        <geometry>
+          <box size="0.4 0.4 0.15"/>
+        </geometry>
+      </collision>
+    </link>
   </xacro:macro>
 </robot>

Commit message: adjust ground plane box collider position

File: ur_description/urdf/inc/ur3e_macro.xacro (robot description, xacro)
@@ -79,5 +79,5 @@
       <parent link="ground_plane_box" />
       <child link = "ground_plane_box_board" />
-      <origin xyz="0.0 0.4 0.325" rpy="0.0 0.0 0.0" />
+      <origin xyz="0.0 0.41 0.325" rpy="0.0 0.0 0.0" />
     </joint>
     <link name="ground_plane_box_board">

File: ur_gazebo/urdf/ur.xacro (robot description, xacro)
@@ -99,5 +99,5 @@
     <parent link="ground_plane_box" />
     <child link = "ground_plane_box_board" />
-    <origin xyz="0.0 0.4 0.325" rpy="0.0 0.0 0.0" />
+    <origin xyz="0.0 0.41 0.325" rpy="0.0 0.0 0.0" />
   </joint>
   <link name="ground_plane_box_board">

Commit message: Support RH-P12-RN gripper
add gripper model to the urdf


add gripper to the URDF


add gripper controllers and handle them from the launch files


add ground plane box to the urdf


use KDL instead of trac ik


clean up changes from chess detector branch


add yaw spawn parameter

File: ur_description/urdf/inc/ur3e_macro.xacro (robot description, xacro)
@@ -40,4 +40,36 @@
       safety_k_position="${safety_k_position}"
     />
+    <!-- world link -->
+    <link name="world"/>
+    <joint name="world_joint" type="fixed">
+      <parent link="world"/>
+      <child link="base_link"/>
+      <origin xyz="0 0 0" rpy="0 0 0"/>
+    </joint>
+    <!-- rh_p12_rn_a -->
+    <xacro:include filename="$(find rh_p12_rn_a_description)/urdf/rh_p12_rn_a.xacro" />
+    <!-- add ground plane box TODO: this should be moved to another xacro -->
+    <joint name="ground_joint" type="fixed">
+      <parent link="world" />
+      <child link = "ground_plane_box" />
+      <origin xyz="0.0 0.0 -0.26" rpy="0.0 0.0 0.0" />
+    </joint>
+    <link name="ground_plane_box">
+      <visual>
+        <origin xyz="0 0 0" rpy="0 0 0"/>
+        <geometry>
+          <box size="1.0 1.0 0.5"/>
+        </geometry>
+        <material name="Grey">
+          <color rgba="0.7 0.7 0.7 1.0"/>
+        </material>
+      </visual>
+      <collision>
+        <origin xyz="0 0 0" rpy="0 0 0"/>
+        <geometry>
+          <box size="1.0 1.0 0.5"/>
+        </geometry>
+      </collision>
+    </link>
   </xacro:macro>
 </robot>

File: ur_gazebo/urdf/ur.xacro (robot description, xacro)
@@ -67,3 +67,28 @@
     <origin xyz="0 0 0" rpy="0 0 0"/>
   </joint>
+  <!-- rh_p12_rn_a -->
+  <xacro:include filename="$(find rh_p12_rn_a_description)/urdf/rh_p12_rn_a.xacro" />
+  <!-- add ground plane box TODO: this should be moved to another xacro -->
+  <joint name="ground_joint" type="fixed">
+    <parent link="world" />
+    <child link = "ground_plane_box" />
+    <origin xyz="0.0 0.0 -0.26" rpy="0.0 0.0 0.0" />
+  </joint>
+  <link name="ground_plane_box">
+    <visual>
+      <origin xyz="0 0 0" rpy="0 0 0"/>
+      <geometry>
+        <box size="1.0 1.0 0.5"/>
+      </geometry>
+      <material name="Grey">
+        <color rgba="0.7 0.7 0.7 1.0"/>
+      </material>
+    </visual>
+    <collision>
+      <origin xyz="0 0 0" rpy="0 0 0"/>
+      <geometry>
+        <box size="1.0 1.0 0.5"/>
+      </geometry>
+    </collision>
+  </link>
 </robot>
